File: SMBee.kicad_pcb (KiCad board)
At the start: 2 copper layers, 42.5 x 57 mm, 18 parts, among them J1 CONN_PIN, J2 CONN_PIN, J3 CONN_PIN, J4 CONN_PIN, J5 CONN_PIN, J6 CONN_PIN, SW1 ALPS_SKRB, U1 PIC10LF322-I/OT

Commit message: 1.1.1 > 1.1.2 Migrate to kicad 6 Add (solder) paste layers Minor DRC fixes
Other:
- net class Default removed
- board text added: "SMBee V1.1.2"
- board text added: "milelo.github.io"
- board text removed: "SMBee V1.1.1"
